File: kicad/e-ink-watch.kicad_pcb (KiCad board)
At the start: 4 copper layers, 40 x 40 mm, 42 parts, among them SW1 BTN1, SW2 BTN2, SW3 BTN3, U1 MDBT50Q-1MV2, U2 BQ25120A

Commit message: Pass-AG: D5 GND tie and east–west 3V3 stitch (#2)
* PCB Pass-AG: record R_SCL rot-90 DRC miss and 0402 +Y pad map.

gpt-6-sol rotation KEEP reverted: KiCad 0402 at 90° puts pad 1 at +Y,
so 3V3 stubs drawn to +Y short SCL. CD in-place stub still promoted
ILIM↔PMID. Board KEEP unchanged (ISET via west only).

Co-authored-by: illiapliukhin <illiapliukhin@users.noreply.github.com>

* PCB Pass-AG: park TS via on west B.Cu elbow after Sol review.

gpt-6-sol's TS park at (108.00, 105.65) overlaps VBAT and ISET. The gated KEEP slides the existing via to the TS B.Cu corner (107.8, 105.65) 0.25/0.15; shorting stays 0, unconnected 10→11. ILIM-only and TS F retract still promote CD/SCL/SDA latents.

Co-authored-by: illiapliukhin <illiapliukhin@users.noreply.github.com>

* PCB Pass-AG: Sol vision loop, combined U2 KEEP shorting 0.

Showed gpt-6-sol annotated F/B maps and 3D of U2, then corrected via size (0.20 at 110.75, not 0.25 at 110.80) and retracted the CD vertical that crossed 3V3. One in-place save moves ILIM, CD, TS stubs, and R_SCL west; DRC shorting stays 0.

Co-authored-by: illiapliukhin <illiapliukhin@users.noreply.github.com>

* Give gpt-6-sol a read-only repo loop for U2 reconnect.

Sol can list, grep, and inspect the board itself instead of a pasted brief. Pocket maps hide B-only pads on F.Cu.

Co-authored-by: illiapliukhin <illiapliukhin@users.noreply.github.com>

* Let Sol browse the repo; KEEP R_SCL 3V3 reconnect.

gpt-6-sol opened the board itself. Its first CD haul onto NC E1 was rejected. The follow-up 3V3 L from R_SCL pad2 DRC-gates with shorting 0 and unc 16→15.

Co-authored-by: illiapliukhin <illiapliukhin@users.noreply.github.com>

* Write each Sol follow-up to its own report file.

Keeps the previous explorer transcript when the next stepwise KEEP round runs.

Co-authored-by: illiapliukhin <illiapliukhin@users.noreply.github.com>

* Tie leftover R_LSCTRL 3V3 stub to the pocket via.

Sol browsed the post-3V3 board, refused CD through the SDA diagonal, an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
Parts:
- moved R_SCL 5.96 mm to (106.5, 110.1), turned to 90 degrees
Routing:
- net 3V3: track 99.7 -> 114.8 mm, vias 25 -> 26
- net GND: track 139.0 -> 140.9 mm, vias 43 -> 44
- net CD: track 5.56 -> 6.39 mm, vias 1 -> 2
- net TS: track 7.87 -> 7.16 mm
- net ILIM: track 8.87 -> 8.37 mm
Changed lines of the file:
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@@
 	(footprint "Resistor_SMD:R_0402_1005Metric"
 		(layer "F.Cu")
-		(at 112.0 107.8)
+		(at 106.5 110.1 90)
 		(descr "Resistor SMD 0402 (1005 Metric), square (rectangular) end terminal, IPC-7351 nominal, (Body size source: IPC-SM-782 page 72, https://www.pcb-3d.com/wordpress/wp-content/uploads/ipc-sm-782a_amendment_1_and_2.pdf), generated with kicad-footprint-generator")
 		(tags "resistor")
@@
 	)
 	(via
-		(at 111.45 105.8)
-		(size 0.5)
-		(drill 0.25)
+		(at 110.75 105.8)
+		(size 0.2)
+		(drill 0.15)
 		(layers "F.Cu" "B.Cu")
 		(net 35)
@@
 	(segment
 		(start 110.6 106.0)
-		(end 111.45 105.8)
+		(end 110.6 106.02)
 		(width 0.15)
 		(layer "F.Cu")
@@
 	)
 	(via
-		(at 110.4 105.65)
-		(size 0.35)
+		(at 107.8 105.65)
+		(size 0.25)
 		(drill 0.15)
 		(layers "F.Cu" "B.Cu")
@@
 	)
 	(segment
-		(start 110.4 105.65)
-		(end 110.4 106.0)
+		(start 111.0 106.0)
+		(end 111.0 106.12)
 		(width 0.1)
 		(layer "F.Cu")
@@
 	)
 	(segment
-		(start 110.4 106.0)
-		(end 111.0 106.0)
+		(start 111.0 106.0)
+		(end 111.0 106.12)
 		(width 0.1)
 		(layer "F.Cu")
@@
 	(segment
 		(start 112.8 108.26)
-		(end 112.8 106.8)
+		(end 112.8 108.41)
 		(width 0.15)
 		(layer "F.Cu")
@@
 	)
 	(segment
-		(start 112.8 106.8)
-		(end 110.6 106.8)
+		(start 110.6 106.8)
+		(end 110.63 106.8)
 		(width 0.15)
 		(layer "F.Cu")
@@
 		(net 1)
 	)
+	(segment
+		(start 106.5 109.59)
+		(end 110.5 109.59)
+		(width 0.12)
+		(layer "F.Cu")
+		(net 2)
+	)
+	(segment
+		(start 110.5 109.59)
+		(end 110.5 108.25)
+		(width 0.12)
+		(layer "F.Cu")
+		(net 2)
+	)
+	(segment
+		(start 110.5 108.25)
+		(end 110.16 108.25)
+		(width 0.12)
+		(layer "F.Cu")
+		(net 2)
+	)
+	(segment
+		(start 112.51 107.8)
+		(end 112.16 107.8)
+		(width 0.2)
+		(layer "F.Cu")
+		(net 2)
+	)
+	(via
+		(at 110.6 106.95)
+		(size 0.25)
+		(drill 0.15)
+		(layers "F.Cu" "B.Cu")
+		(net 32)
+	)
+	(segment
+		(start 110.6 106.8)
+		(end 110.6 106.95)
+		(width 0.15)
+		(layer "F.Cu")
+		(net 32)
+	)
+	(segment
+		(start 110.6 106.95)
+		(end 112.65 106.95)
+		(width 0.12)
+		(layer "B.Cu")
+		(net 32)
+	)
+	(segment
+		(start 112.65 106.95)
+		(end 112.65 108.41)
+		(width 0.12)
+		(layer "B.Cu")
+		(net 32)
+	)
+	(segment
+		(start 112.65 108.41)
+		(end 113.3 108.41)
+		(width 0.12)
+		(layer "B.Cu")
+		(net 32)
+	)
+	(segment
+		(start 110.6 106.0)
+		(end 110.75 106.0)
+		(width 0.08)
+		(layer "F.Cu")
+		(net 35)
+	)
+	(segment
+		(start 110.75 106.0)
+		(end 110.75 105.8)
+		(width 0.08)
+		(layer "F.Cu")
+		(net 35)
+	)
+	(via
+		(at 112.4 106.55)
+		(size 0.25)
+		(drill 0.15)
+		(layers "F.Cu" "B.Cu")
+		(net 1)
+	)
+	(segment
+		(start 111.8 106.4)
+		(end 112.4 106.4)
+		(width 0.12)
+		(layer "F.Cu")
+		(net 1)
+	)
+	(segment
+		(start 112.4 106.4)
+		(end 112.4 106.55)
+		(width 0.12)
+		(layer "F.Cu")
+		(net 1)
+	)
+	(segment
+		(start 112.4 106.55)
+		(end 112.8 106.55)
+		(width 0.12)
+		(layer "F.Cu")
+		(net 1)
+	)
+	(segment
+		(start 112.8 106.55)
+		(end 112.8 107.24)
+		(width 0.12)
+		(layer "F.Cu")
+		(net 1)
+	)
+	(via
+		(at 110.4 108.25)
+		(size 0.25)
+		(drill 0.15)
+		(layers "F.Cu" "B.Cu")
+		(net 2)
+	)
+	(segment
+		(start 110.4 108.25)
+		(end 110.4 108.55)
+		(width 0.12)
+		(layer "B.Cu")
+		(net 2)
+	)
+	(segment
+		(start 110.4 108.55)
+		(end 102.52 108.55)
+		(width 0.12)
+		(layer "B.Cu")
+		(net 2)
+	)
+	(segment
+		(start 102.52 108.55)
+		(end 102.52 109.4)
+		(width 0.12)
+		(layer "B.Cu")
+		(net 2)
+	)
 	(via
